File: src_files/HallCoinDetector/HallCoinDetector.kicad_pcb (KiCad board)
At the start: 2 copper layers, 30.5 x 22.9 mm, 30 parts, among them M1 Motor_DC 3V, Q2 BSS214NW, U1 SE555D, U2 TPS61070, U3 49E Hall, U4 LM393

Commit message: delete backups
Parts:
- moved U3 2.75 mm to (108.2, 118.1)
Changed lines of the file:
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@@
   )
   (footprint "Package_TO_SOT_THT:TO-92_Inline_W4.0mm_Horizontal_FlatSideDown" (layer "F.Cu")
-    (at 109.22 115.57 -90)
+    (at 108.21 118.1275 -90)
     (descr "TO-92 horizontal, leads in-line, narrow, oval pads, drill 0.75mm (see NXP sot054_po.pdf)")
     (tags "to-92 sc-43 sc-43a sot54 PA33 transistor")

Commit message: diseño de librerias y ubicación de componentes
Parts:
- added SW1: On, Button_Switch_SMD:SW_SPDT_PCM12, B.Cu at (173.2, 103.8)
- BT1: footprint Battery:BatteryHolder_Keystone_3002_1x2032 -> Batery Holder:cr1616
- U3: moved to B.Cu
- moved R2 96.5 mm to (178.6, 112.4), turned to 90 degrees
- moved R1 94.8 mm to (176.5, 112.4), turned to -90 degrees
- moved U4 91.6 mm to (189.2, 111.8)
- moved U1 91.6 mm to (189.2, 102.9), turned to 90 degrees
- moved C5 81.4 mm to (185.1, 118.7)
- moved C2 74.6 mm to (178.6, 108.9), turned to 90 degrees
- moved C1 72.6 mm to (176.5, 105.3), turned to -90 degrees
- moved C3 72.5 mm to (176.5, 108.9), turned to 90 degrees
- moved U2 65.7 mm to (173.2, 111.4)
- moved Q2 64.1 mm to (169.3, 123.0)
- moved L1 63.8 mm to (172.9, 106.7)
- moved U3 62.2 mm to (165.8, 94.4), turned to 0 degrees
- moved R14 19.4 mm to (110.2, 111.8)
- moved D3 8.78 mm to (123.8, 91.4)
- moved BT1 6.90 mm to (158.3, 113.2), turned to 90 degrees
Connections:
- BT1 pad 1: /BAT -> Net-(BT1-+)

Commit message: delete backups
Parts:
- C4, C5, R10, R11, R3, R4, R5, R6, R7, R8, R9, U1, U4, r12: moved to B.Cu
- D3: footprint Diode_SMD:D_SOD-323 -> Diode_SMD:D_SOD-123; moved to B.Cu
- U3: footprint Package_TO_SOT_THT:TO-92_Inline_W4.0mm_Horizontal_FlatSideDown -> Package_TO_SOT_SMD:SOT-23-3
- moved R3 84.5 mm to (166.8, 104.5), turned to -90 degrees
- moved R7 83.1 mm to (169.8, 107.3)
- moved R8 83.1 mm to (169.8, 109.2), turned to 180 degrees
- moved R4 80.5 mm to (162.7, 105.5), turned to 180 degrees
- moved r12 76.6 mm to (167.7, 113.0)
- moved R5 76.3 mm to (158.4, 108.9)
- moved R13 74.6 mm to (164.2, 119.8), turned to -90 degrees
- moved R6 71.8 mm to (158.4, 106.9)
- moved R10 71.8 mm to (158.5, 115.3), turned to 180 degrees
- moved R9 71.7 mm to (158.4, 113.4), turned to 180 degrees
- moved M1 69.1 mm to (172.8, 121.9)
- moved R11 67.9 mm to (158.4, 111.2)
- moved D3 57.4 mm to (175.7, 115.8)
- moved R14 56.6 mm to (166.3, 119.8), turned to 90 degrees
- moved C4 49.9 mm to (158.3, 119.4), turned to 180 degrees
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Connections:
- BT1 pad 1: Net-(BT1-+) -> /BAT
- C1 pad 1: /BAT -> /3V
- D3 pad 1: /BAT -> /3V
- L1 pad 1: /BAT -> /3V
- M1 pad 1: /BAT -> /3V
- SW1 pad 1: /BAT -> /3V
- SW1 pad 2: /BAT -> /3V
- SW1 pad 3: Net-(BT1-+) -> /BAT
- U2 pad 3: /BAT -> /3V
- U2 pad 6: /BAT -> /3V
Routing:
- net /+5V: track 0.00 -> 25.0 mm, vias 0 -> 1
- net /3V: track 0.00 -> 13.2 mm
- net Net-(U1-R): track 0.00 -> 11.4 mm
- net Net-(U1-THR): track 0.00 -> 11.0 mm
- net Net-(U4A-+): track 0.00 -> 7.56 mm
- net Net-(U1-DIS): track 0.00 -> 5.58 mm
- net Net-(U4B-+): track 0.00 -> 5.12 mm
- net Net-(U4A--): track 0.00 -> 4.97 mm
- net Net-(U2-SW): track 0.00 -> 4.95 mm
- net Net-(U2-FB): track 0.00 -> 4.65 mm
- net Net-(U1-CV): track 0.00 -> 3.10 mm
- net Net-(D1-A): track 0.00 -> 2.54 mm
- net Net-(U4B--): track 0.00 -> 2.43 mm
- net Net-(U3-OUT): track 0.00 -> 1.93 mm
- added copper zone on B.Cu, net /3V
- added copper zone on F.Cu, net /3V

Commit message: first_delivery
Parts:
- D1, D2: footprint Diode_THT:D_DO-35_SOD27_P7.62mm_Horizontal -> Diode_SMD:D_0805_2012Metric; moved to B.Cu
- R13: moved to B.Cu
- moved D2 59.8 mm to (165.6, 121.3), turned to 90 degrees
- moved D1 56.5 mm to (161.0, 121.5), turned to 180 degrees
- moved C2 11.8 mm to (167.8, 103.9), turned to 0 degrees
- moved M1 5.03 mm to (167.7, 122.0), turned to 180 degrees
- moved R4 4.26 mm to (166.8, 104.5), turned to 90 degrees
- moved R14 2.95 mm to (163.8, 121.4)
- moved R3 2.88 mm to (164.1, 105.5), turned to 0 degrees
- moved Q2 2.15 mm to (167.8, 117.8), turned to -90 degrees
- moved R13 1.62 mm to (163.7, 121.3), turned to 90 degrees
- moved D3 1.54 mm to (176.3, 114.4), turned to 180 degrees
- moved C1 1.32 mm to (177.2, 107.2)
- moved R6 1.17 mm to (159.6, 107.0), turned to -90 degrees
- moved R5 0.92 mm to (157.5, 108.8), turned to 90 degrees
- moved C3 0.76 mm to (177.2, 109.3), turned to 0 degrees
- moved R2 0.50 mm to (178.2, 112.0)
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Connections:
- SW1 pad 1: /3V -> /BAT
- SW1 pad 2: /3V -> /BAT
- SW1 pad 3: /BAT -> /3V
Routing:
- net /BAT: track 0.00 -> 45.4 mm, vias 0 -> 1
- net /+5V: track 25.0 -> 50.1 mm, vias 1 -> 5
- net Net-(D1-A): track 2.54 -> 25.8 mm
- net /3V: track 13.2 -> 34.9 mm, vias 0 -> 1
- net Net-(D3-A): track 0.00 -> 10.3 mm, vias 0 -> 1
- net Net-(Q2-G): track 0.00 -> 6.28 mm
- net Net-(D1-K): track 0.00 -> 6.24 mm, vias 0 -> 1
- net Net-(D2-A): track 0.00 -> 4.09 mm
- net Net-(U3-OUT): track 1.93 -> 4.71 mm
- net Net-(U4B-+): track 5.12 -> 3.68 mm
- net Net-(U4A--): track 4.97 -> 5.64 mm
- net Net-(U2-FB): track 4.65 -> 4.10 mm
- net GND: vias 0 -> 10
- added copper zone on B.Cu, net GND
- added copper zone on F.Cu, net GND
- removed copper zone on B.Cu, net /3V
- removed copper zone on F.Cu, net /3V
